Commit message: Made a basic hand coded forklift similar to the Cangozpi forklift. Nothing functional yet.

File: urdf/warehouse_bot.urdf (robot description, URDF)
Before this commit: robot warehouse_bot, 6 links, 5 joints
Links:
- added link body_link, mass 50.0; collision box size=1.6 1.1 0.5; visual box size=1.6 1.1 0.5
- added link left_fork_link, mass 1.0; collision box size=1 0.1 0.05; visual box size=1 0.1 0.05
- added link rails_link, mass 5.0; collision box size=0.1 1.1 1.5; visual box size=0.1 1.1 1.5
- added link rails_plate_link, mass 5.0; collision box size=0.1 1.1 0.5; visual box size=0.1 1.1 0.5
- added link right_fork_link, mass 1.0; collision box size=1 0.1 0.05; visual box size=1 0.1 0.05
- link base_link: geometry collision box size=1.6 1.1 0.15; visual box size=1.6 1.1 0.15
- link caster_wheel: geometry collision sphere radius=0.1; visual sphere radius=0.1
- link left_wheel: geometry collision cylinder length=0.05 radius=0.2; visual cylinder length=0.05 radius=0.2
- link right_wheel: geometry collision cylinder length=0.05 radius=0.2; visual cylinder length=0.05 radius=0.2
Joints:
- added joint base_body_joint: type fixed, parent base_link, child body_link, origin xyz=0 0 0.35
- added joint body_rails_joint: type fixed, parent body_link, child rails_link, origin xyz=0.85 0 0.5
- added joint rails_plate_left_fork_joint: type fixed, parent rails_plate_link, child left_fork_link, origin xyz=0.55 -0.3 -0.225
- added joint rails_plate_right_fork_joint: type fixed, parent rails_plate_link, child right_fork_link, origin xyz=0.55 0.3 -0.225
- added joint rails_rails_plate_joint: type fixed, parent rails_link, child rails_plate_link, origin xyz=0.1 0 -0.675
- joint caster_wheel_joint: origin xyz=0.2 0 -0.1 -> xyz=-0.75 0 -0.15
- joint left_wheel_joint: origin xyz=-0.2 0.175 -0.05 rpy=-1.5708 0 0 -> xyz=0.55 0.575 -0.05 rpy=-1.5708 0 0
- joint right_wheel_joint: origin xyz=-0.2 -0.175 -0.05 rpy=-1.5708 0 0 -> xyz=0.55 -0.575 -0.05 rpy=-1.5708 0 0

Commit message: Basic forklift structure done along with lidar and camera placement. Forks don't move yet.

File: urdf/warehouse_bot.urdf (robot description, URDF)
Before this commit: robot warehouse_bot, 11 links, 10 joints
Links:
- link lidar: geometry collision cylinder length=0.05 radius=0.05; visual cylinder length=0.05 radius=0.05
Joints:
- joint camera_joint: origin xyz=0.27 0 0.01 rpy=0 0 0 -> xyz=0.05 0 0.7 rpy=0 0 0; parent base_link -> rails_link
- joint lidar_joint: origin xyz=0 0 0.1 rpy=0 0 0 -> xyz=0 0 0.775 rpy=0 0 0; parent base_link -> rails_link

Commit message: Working on getting Nav2 to run.  Fixed map transform errors in RViz. Mapping not working yet.

File: urdf/warehouse_bot.urdf (robot description, URDF)
Before this commit: robot warehouse_bot, 11 links, 10 joints
Links:
- added link base_footprint, mass 5.0; collision box size=1.6 1.1 0.15; visual box size=1.6 1.1 0.15
- link base_link: mass 5.0 -> None; geometry 
Joints:
- added joint base_footprint_joint: type fixed, parent base_link, child base_footprint, origin xyz=0 0 -0.05
